File: Hardware/tornado-Backplane.sch (EAGLE design)
At the start: 13 parts, among them CON1 ROV_SHIELD_V2

Commit message: Wrapping up initial board layout
Connections:
- removed net N$23: CON1G$1.P$14
- new net SONAR_TIMER: BRICKS_COM.C2, CON1G$1.P$14
Changed lines of the file:
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@@
 <?xml version="1.0" encoding="utf-8"?>
 <!DOCTYPE eagle SYSTEM "eagle.dtd">
-<eagle version="7.6.0">
+<eagle version="6.6.0">
 <drawing>
 <settings>
@@
 </segment>
 </net>
-<net name="N$23" class="0">
-<segment>
-<pinref part="CON1" gate="G$1" pin="P$14"/>
-<wire x1="431.8" y1="-86.36" x2="439.42" y2="-86.36" width="0.1524" layer="91"/>
-</segment>
-</net>
 <net name="N$24" class="0">
 <segment>
@@
 <pinref part="CON1" gate="G$1" pin="P$15"/>
 <wire x1="431.8" y1="-91.44" x2="439.42" y2="-91.44" width="0.1524" layer="91"/>
+<label x="434.34" y="-91.44" size="1.778" layer="95"/>
 </segment>
 </net>
@@
 </segment>
 </net>
+<net name="SONAR_TIMER" class="0">
+<segment>
+<pinref part="BRICKS_COM" gate="G$1" pin="C2"/>
+<wire x1="228.6" y1="-60.96" x2="238.76" y2="-60.96" width="0.1524" layer="91"/>
+<label x="231.14" y="-60.96" size="1.778" layer="95"/>
+</segment>
+<segment>
+<pinref part="CON1" gate="G$1" pin="P$14"/>
+<wire x1="431.8" y1="-86.36" x2="439.42" y2="-86.36" width="0.1524" layer="91"/>
+<label x="434.34" y="-86.36" size="1.778" layer="95"/>
+</segment>
+</net>

Commit message: Fixes from Michael
Mostly layout, fixing ground islands, and other small fixes.
Parts:
- gave numbers to parts that had none: 1
Changed lines of the file:
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@@
 <?xml version="1.0" encoding="utf-8"?>
 <!DOCTYPE eagle SYSTEM "eagle.dtd">
-<eagle version="6.6.0">
+<eagle version="7.6.0">
 <drawing>
 <settings>
@@
 <part name="FRAME3" library="frames" deviceset="FRAME_A_L" device=""/>
 <part name="FRAME4" library="frames" deviceset="FRAME_A_L" device=""/>
-<part name="IO_PUMP?" library="Connectors" deviceset="MICRO-FIT-4-SMD" device="" technology="-PART"/>
+<part name="IO_PUMP" library="Connectors" deviceset="MICRO-FIT-4-SMD" device="" technology="-PART"/>
 <part name="SOLENOID_SWITCH" library="Connectors" deviceset="MICRO-FIT-4-SMD" device="" technology="-PART"/>
 <part name="EMPTY" library="Connectors" deviceset="MICRO-FIT-4-SMD" device="" technology="-PART"/>
@@
 <instance part="FRAME4" gate="G$1" x="0" y="-215.9"/>
 <instance part="FRAME4" gate="G$2" x="172.72" y="-215.9"/>
-<instance part="IO_PUMP?" gate="G$1" x="68.58" y="-167.64" rot="R90"/>
+<instance part="IO_PUMP" gate="G$1" x="68.58" y="-167.64" rot="R90"/>
 <instance part="SOLENOID_SWITCH" gate="G$1" x="139.7" y="-43.18" rot="R90"/>
 <instance part="EMPTY" gate="G$1" x="139.7" y="-60.96" rot="R90"/>
@@
 </segment>
 <segment>
-<pinref part="IO_PUMP?" gate="G$1" pin="C1"/>
+<pinref part="IO_PUMP" gate="G$1" pin="C1"/>
 <wire x1="76.2" y1="-170.18" x2="96.52" y2="-170.18" width="0.1524" layer="91"/>
 <label x="78.74" y="-170.18" size="1.9304" layer="95"/>
@@
 </segment>
 <segment>
-<pinref part="IO_PUMP?" gate="G$1" pin="C3"/>
+<pinref part="IO_PUMP" gate="G$1" pin="C3"/>
 <wire x1="76.2" y1="-165.1" x2="96.52" y2="-165.1" width="0.1524" layer="91"/>
 <label x="78.74" y="-165.1" size="1.778" layer="95"/>
@@
 </segment>
 <segment>
-<pinref part="IO_PUMP?" gate="G$1" pin="C4"/>
+<pinref part="IO_PUMP" gate="G$1" pin="C4"/>
 <wire x1="76.2" y1="-162.56" x2="96.52" y2="-162.56" width="0.1524" layer="91"/>
 <label x="78.74" y="-162.56" size="1.778" layer="95"/>
@@
 <net name="GPIO" class="0">
 <segment>
-<pinref part="IO_PUMP?" gate="G$1" pin="C2"/>
+<pinref part="IO_PUMP" gate="G$1" pin="C2"/>
 <wire x1="76.2" y1="-167.64" x2="96.52" y2="-167.64" width="0.1524" layer="91"/>
 <label x="78.74" y="-167.64" size="1.778" layer="95"/>
