File: Hardware/tornado-shield.sch (EAGLE design)
At the start: 30 parts, among them CON1 ROV_SHIELD_V2, Q1 DMP2012SN-7, U1 LM2678S-5.0, U2 LM3409HV'LM3409HV'

Commit message: Continued to finish Shield
Still needs Pi Pinout
Connections:
- removed net V_IN: C_F.1, C_IN1.1, C_IN2.1, R_SNS.2, R_UV2.2, U2.CSP, U2.VIN
- removed net V_OUT: L2.2, R_OFF.1
- new net LED_CON: R_PD.1
- net +12V: now also C_F.1, C_IN1.1, C_IN2.1, R_SNS.2, R_UV2.2, U2.CSP, U2.VIN
- net LED_PWM: now also L2.2, R_OFF.1; no longer R_PD.1
Other:
- note added: "LED DRIVER"
- note added: "Linear Reg"
- note added: "Ras-Pi"
- note added: "SOL DRIVER"

Commit message: Wrapping up initial board layout
Parts:
- added RPD, RPD1: 1k, DiscreteComponents:R-US_R0603
Connections:
- removed net LED_PMW: CON1G$1.P$18
- removed net N$23: CON1G$1.P$14
- removed net SCL: CON1G$1.P$20
- removed net SDA: CON1G$1.P$22
- new net +3V3: U$2.3V3@1
- new net SONAR_TIMER: CON1G$1.P$14, U$2.#16
- net GND: now also RPD.1, RPD1.1
- net GPIO: now also U$2.#4
- net GPIO2: now also U$2.#17
- net GPIO3: now also U$2.#27
- net GPIO4: now also U$2.#22
- net GPIO5: now also U$2.#6
- net GPIO6: now also U$2.#20
- net GPIO7: now also U$2.#21
- net LED_CON: now also U$2.#13
- net NAV_SCL: now also CON1G$1.P$20
- net NAV_SDA: now also CON1G$1.P$22
- net SOL1_IN: now also RPD1.2, U$2.#19
- net SOL2_IN: now also RPD.2, U$2.#26
- net SONAR_PWM: now also U$2.#12
Other:
- moved on the sheet: U$5

Commit message: Board Design Rev 1.0
Connections:
- removed net KJ: CON1G$2.P$17
- removed net N$10: CON1G$1.P$1
- removed net N$11: CON1G$2.P$18
- removed net N$24: CON1G$1.P$13
- removed net N$25: CON1G$1.P$12
- removed net N$26: CON1G$1.P$11
- removed net N$27: CON1G$1.P$10
- removed net N$28: CON1G$1.P$9
- removed net N$29: CON1G$1.P$8
- removed net N$30: CON1G$1.P$7
- removed net N$31: CON1G$1.P$6
- removed net N$32: CON1G$1.P$5
- removed net N$33: CON1G$1.P$4
- removed net N$34: CON1G$1.P$3
- removed net N$37: CON1G$2.P$16
- removed net N$38: CON1G$2.P$15
- removed net N$39: CON1G$2.P$14
- removed net N$40: CON1G$2.P$13
- removed net N$41: CON1G$2.P$12
- removed net N$42: CON1G$2.P$11
- removed net N$43: CON1G$2.P$10
- removed net N$44: CON1G$2.P$9
- removed net N$45: CON1G$2.P$8
- removed net N$46: CON1G$2.P$7
- removed net N$47: CON1G$2.P$6
- removed net N$48: CON1G$2.P$5
- removed net N$49: CON1G$2.P$4
- removed net N$50: CON1G$2.P$3
- removed net N$6: U$2.GND@1
- removed net N$9: CON1G$1.P$2
- net GND: now also U$2.GND@1
Other:
- moved on the sheet: C2, C3, L1, U$3

Commit message: Fixes from Michael
Mostly layout, fixing ground islands, and other small fixes.
Other:
- note added: "Buck Converter"
- note removed: "Linear Reg"
Changed lines of the file:
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@@
 <text x="180.34" y="160.02" size="1.778" layer="97">Ras-Pi</text>
 <text x="180.34" y="160.02" size="1.778" layer="97">Ras-Pi</text>
-<text x="175.26" y="86.36" size="1.778" layer="97">Linear Reg</text>
+<text x="175.26" y="86.36" size="1.778" layer="97">Buck Converter</text>
 <text x="345.44" y="223.52" size="1.778" layer="97">SOL DRIVER</text>
 <text x="345.44" y="223.52" size="1.778" layer="97">SOL DRIVER</text>

Commit message: Added Status LEDs for power and Solenoids
Parts:
- added PWR_ON, SOL1_STAT, SOL2_STAT: (no value), eagle-ltspice:LED_ESML0603
- added R3, R4, R5: (no value), rcl:R-US_R0603
- R1, R2: device rcl:R-US_R1206 -> rcl:R-US_R0603
Connections:
- new net N$12: PWR_ON.C, R5.2
- new net N$9: R4.2, SOL1_STAT.C
- new net SOL2_STAT: R3.2, SOL2_STAT.C
- net +5V: now also PWR_ON.A
- net GND: now also R3.1, R4.1, R5.1
- net SOL_O1: now also SOL1_STAT.A
- net SOL_O2: now also SOL2_STAT.A
Changed lines of the file:
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@@
 <part name="U$4" library="samssuperhot" deviceset="SK1545-TP" device=""/>
 <part name="U$5" library="samssuperhot" deviceset="SK1545-TP" device=""/>
-<part name="R2" library="rcl" deviceset="R-US_" device="R1206"/>
-<part name="R1" library="rcl" deviceset="R-US_" device="R1206"/>
+<part name="R2" library="rcl" deviceset="R-US_" device="R0603"/>
+<part name="R1" library="rcl" deviceset="R-US_" device="R0603"/>
 <part name="GND4" library="supply1" deviceset="GND" device=""/>
 <part name="GND5" library="supply1" deviceset="GND" device=""/>
@@
 <part name="GND17" library="supply1" deviceset="GND" device=""/>
 <part name="GND18" library="supply1" deviceset="GND" device=""/>
+<part name="PWR_ON" library="eagle-ltspice" deviceset="LED_E" device="SML0603"/>
+<part name="SOL1_STAT" library="eagle-ltspice" deviceset="LED_E" device="SML0603"/>
+<part name="SOL2_STAT" library="eagle-ltspice" deviceset="LED_E" device="SML0603"/>
+<part name="GND19" library="supply1" deviceset="GND" device=""/>
+<part name="GND20" library="supply1" deviceset="GND" device=""/>
+<part name="GND21" library="supply1" deviceset="GND" device=""/>
+<part name="R3" library="rcl" deviceset="R-US_" device="R0603"/>
+<part name="R4" library="rcl" deviceset="R-US_" device="R0603"/>
+<part name="R5" library="rcl" deviceset="R-US_" device="R0603"/>
 </parts>
 <sheets>
@@
 <instance part="GND17" gate="1" x="213.36" y="122.936"/>
 <instance part="GND18" gate="1" x="197.104" y="143.764"/>
+<instance part="PWR_ON" gate="G$1" x="264.16" y="71.12"/>
+<instance part="SOL1_STAT" gate="G$1" x="281.94" y="203.2"/>
+<instance part="SOL2_STAT" gate="G$1" x="304.8" y="180.34"/>
+<instance part="GND19" gate="1" x="281.94" y="185.42"/>
+<instance part="GND20" gate="1" x="304.8" y="160.02"/>
+<instance part="GND21" gate="1" x="264.16" y="48.26"/>
+<instance part="R3" gate="G$1" x="304.8" y="167.64" rot="R90"/>
+<instance part="R4" gate="G$1" x="281.94" y="193.04" rot="R90"/>
+<instance part="R5" gate="G$1" x="264.16" y="58.42" rot="R90"/>
 </instances>
 <busses>
@@
 <wire x1="193.04" y1="146.05" x2="197.104" y2="146.05" width="0.1524" layer="91"/>
 <pinref part="GND18" gate="1" pin="GND"/>
+</segment>
+<segment>
+<pinref part="GND21" gate="1" pin="GND"/>
+<wire x1="264.16" y1="50.8" x2="264.16" y2="53.34" width="0.1524" layer="91"/>
+<pinref part="R5" gate="G$1" pin="1"/>
+</segment>
+<segment>
+<pinref part="GND20" gate="1" pin="GND"/>
+<pinref part="R3" gate="G$1" pin="1"/>
+</segment>
+<segment>
+<pinref part="GND19" gate="1" pin="GND"/>
+<pinref part="R4" gate="G$1" pin="1"/>
 </segment>
 </net>
@@
 <junction x="241.3" y="76.2"/>
 <pinref part="P+5" gate="1" pin="+5V"/>
+<pinref part="PWR_ON" gate="G$1" pin="A"/>
+<wire x1="248.92" y1="76.2" x2="264.16" y2="76.2" width="0.1524" layer="91"/>
+<wire x1="264.16" y1="76.2" x2="264.16" y2="73.66" width="0.1524" layer="91"/>
+<junction x="248.92" y="76.2"/>
 </segment>
 <segment>
@@
 <junction x="337.82" y="208.28"/>
 <label x="299.72" y="208.28" size="1.778" layer="95"/>
-<wire x1="322.58" y1="208.28" x2="299.72" y2="208.28" width="0.1524" layer="91"/>
+<wire x1="322.58" y1="208.28" x2="281.94" y2="208.28" width="0.1524" layer="91"/>
 <junction x="322.58" y="208.28"/>
+<pinref part="SOL1_STAT" gate="G$1" pin="A"/>
+<wire x1="281.94" y1="205.74" x2="281.94" y2="208.28" width="0.1524" layer="91"/>
 </segment>
 </net>
@@
 <label x="297.18" y="187.96" size="1.778" layer="95"/>
 <pinref part="R2" gate="G$1" pin="2"/>
-<wire x1="320.04" y1="187.96" x2="297.18" y2="187.96" width="0.1524" layer="91"/>
+<wire x1="320.04" y1="187.96" x2="304.8" y2="187.96" width="0.1524" layer="91"/>
 <junction x="320.04" y="187.96"/>
+<pinref part="SOL2_STAT" gate="G$1" pin="A"/>
+<wire x1="304.8" y1="187.96" x2="297.18" y2="187.96" width="0.1524" layer="91"/>
+<wire x1="304.8" y1="182.88" x2="304.8" y2="187.96" width="0.1524" layer="91"/>
+<junction x="304.8" y="187.96"/>
 </segment>
 </net>
@@
 </segment>
 </net>
+<net name="SOL2_STAT" class="0">
+<segment>
+<pinref part="SOL2_STAT" gate="G$1" pin="C"/>
+<wire x1="304.8" y1="175.26" x2="304.8" y2="172.72" width="0.1524" layer="91"/>
+<pinref part="R3" gate="G$1" pin="2"/>
+</segment>
+</net>
+<net name="N$12" class="0">
+<segment>
+<pinref part="PWR_ON" gate="G$1" pin="C"/>
+<wire x1="264.16" y1="63.5" x2="264.16" y2="66.04" width="0.1524" layer="91"/>
+<pinref part="R5" gate="G$1" pin="2"/>
+</segment>
+</net>
+<net name="N$9" class="0">
+<segment>
+<pinref part="SOL1_STAT" gate="G$1" pin="C"/>
+<pinref part="R4" gate="G$1" pin="2"/>
+</segment>
+</net>
